File: weather_station_sensor_board.kicad_pcb (KiCad board)
At the start: 2 copper layers, 56 x 51 mm, 11 parts, among them J1 Conn_01x04, J2 Conn_01x04, J3 Conn_01x04, J4 Conn_01x05, J5 Conn_01x02, M1 MountingHole_2.2mm_M2_Pad_Via, M2 MountingHole_2.2mm_M2_Pad_Via, M3 MountingHole_2.2mm_M2_Pad_Via, M4 MountingHole_2.2mm_M2_Pad_Via, U1 MAX3490xPA

Commit message: Added silscreen annotation for headers
Routing:
- net RX: track 31.1 -> 73.4 mm
- net TX: track 34.7 -> 71.0 mm
- net +3V3: track 118.9 -> 86.8 mm
- net RX_NEG: track 13.6 -> 17.3 mm
- net TX_NEG: track 15.5 -> 18.1 mm
- net TX_POS: track 17.3 -> 18.8 mm
- net RX_POS: track 10.8 -> 11.5 mm
- net GND: vias 37 -> 33
Other:
- board text added: "+3V3"
- board text added: "+5V"
- board text added: "Feather M0"
- board text added: "GND"
- board text added: "MAX3490"
- board text added: "RX"
- board text added: "SCL"
- board text added: "SDA"
- board text added: "TX"
- board text added: "~{RX}"
- board text added: "~{TX}"
