File: weather_station_sensor_board.kicad_pcb (KiCad board)
At the start: 2 copper layers, 56 x 51 mm, 11 parts, among them J1 Conn_01x04, J2 Conn_01x04, J3 Conn_01x04, J4 Conn_01x05, J5 Conn_01x02, M1 MountingHole_2.2mm_M2_Pad_Via, M2 MountingHole_2.2mm_M2_Pad_Via, M3 MountingHole_2.2mm_M2_Pad_Via, M4 MountingHole_2.2mm_M2_Pad_Via, U1 MAX3490xPA

Commit message: rev 2.0
Parts:
- added J6: Conn_01x02, Connector_PinHeader_2.54mm:PinHeader_1x02_P2.54mm_Vertical, F.Cu at (121.9, 63.5)
- moved J5 20.5 mm to (121.9, 73.7)
- moved U1 15.2 mm to (111.8, 76.2)
- moved J1 5.68 mm to (129.5, 73.7)
- moved J2 5.68 mm to (129.5, 68.6)
- moved J3 5.68 mm to (129.5, 63.5)
- moved J4 5.68 mm to (104.1, 63.5)
- moved M2 5.00 mm to (143.0, 61.6)
- moved M4 5.00 mm to (143.0, 106.7)
Connections:
- A1 pad 24: unconnected-(A1-D12-Pad24) -> D1
Routing:
- net D1: track 0.00 -> 20.4 mm
- net +3V3: track 86.8 -> 74.5 mm
- net TX_POS: track 18.8 -> 6.88 mm
- net TX: track 71.0 -> 78.9 mm
- net RX: track 73.4 -> 81.0 mm
- net TX_NEG: track 18.1 -> 10.5 mm
- net RX_POS: track 11.5 -> 18.4 mm
- net RX_NEG: track 17.3 -> 14.1 mm
- net SCL: track 16.3 -> 18.8 mm
- net SDA: track 16.3 -> 18.8 mm
- net +5V: track 14.8 -> 13.8 mm
- net GND: vias 33 -> 49
Other:
- board size 56 x 51 mm -> 51 x 51 mm
- board text added: "3V3"
- board text added: "5V"
- board text added: "D1"
- board text added: "Weather Station Sensor Board Rev 2.0"
- board text removed: "+3V3"
- board text removed: "+5V"
- board text removed: "Weather Station Sensor Board Rev 1.0"
