File: weather_station_sensor_board.kicad_sch (KiCad schematic)
At the start: 7 parts, among them J1 Conn_01x04, J2 Conn_01x04, J3 Conn_01x04, J4 Conn_01x05, J5 Conn_01x02, U1 MAX3490xPA

Commit message: rev 2.0
Parts:
- added J6: Conn_01x02, Connector_PinHeader_2.54mm:PinHeader_1x02_P2.54mm_Vertical, symbol Connector_Generic:Conn_01x02
Connections:
- net GND: now also J6.1 (Pin_1)
- net D1: now reaches A1.24 (D12)
- net D1: now also J6.2 (Pin_2)
- no-connect marks 20 -> 19
Changed lines of the file:
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@@
   (title_block
     (title "Weather Station Sensor Board")
-    (date "2024-01-30")
-    (rev "REV 1.0")
+    (date "2024-01-31")
+    (rev "REV 2.0")
     (company "Flavian Kaufmann")
   )
@@
   (no_connect (at 100.33 85.09))
   (no_connect (at 125.73 105.41))
-  (no_connect (at 100.33 95.25))
   (no_connect (at 125.73 92.71))
   (no_connect (at 125.73 110.49))
@@
     (stroke (width 0) (type default))
   )
+  (wire (pts (xy 208.915 68.58) (xy 208.915 72.39))
+    (stroke (width 0) (type default))
+  )
   (wire (pts (xy 170.18 68.58) (xy 170.18 72.39))
     (stroke (width 0) (type default))
@@
     (stroke (width 0) (type default))
   )
+  (wire (pts (xy 206.375 64.77) (xy 206.375 72.39))
+    (stroke (width 0) (type default))
+  )
   (wire (pts (xy 200.66 68.58) (xy 200.66 72.39))
     (stroke (width 0) (type default))
@@
   )
   (wire (pts (xy 176.53 64.77) (xy 176.53 72.39))
+    (stroke (width 0) (type default))
+  )
+  (wire (pts (xy 96.52 95.25) (xy 100.33 95.25))
     (stroke (width 0) (type default))
   )
@@
     )
   )
+  (global_label "D1" (shape input) (at 96.52 95.25 180) (fields_autoplaced)
+    (effects (font (size 1.27 1.27)) (justify right))
+    (property "Intersheetrefs" "${INTERSHEET_REFS}" (at 91.0553 95.25 0)
+      (effects (font (size 1.27 1.27)) (justify right) hide)
+    )
+  )
   (global_label "SCL" (shape input) (at 96.52 125.73 180) (fields_autoplaced)
     (effects (font (size 1.27 1.27)) (justify right))
@@
     (effects (font (size 1.27 1.27)) (justify left))
     (property "Intersheetrefs" "${INTERSHEET_REFS}" (at 151.13 58.2772 90)
+      (effects (font (size 1.27 1.27)) (justify left) hide)
+    )
+  )
+  (global_label "D1" (shape input) (at 206.375 64.77 90) (fields_autoplaced)
+    (effects (font (size 1.27 1.27)) (justify left))
+    (property "Intersheetrefs" "${INTERSHEET_REFS}" (at 206.375 59.3053 90)
       (effects (font (size 1.27 1.27)) (justify left) hide)
     )
@@
     )
   )
+  (symbol (lib_id "Connector_Generic:Conn_01x02") (at 208.915 77.47 270) (unit 1)
+    (in_bom yes) (on_board yes) (dnp no)
+    (property "Reference" "J6" (at 206.375 81.28 90)
+      (effects (font (size 1.27 1.27)) (justify left))
+    )
+    (property "Value" "Conn_01x02" (at 203.2 83.82 90)
+      (effects (font (size 1.27 1.27)) (justify left))
+    )
+    (property "Footprint" "Connector_PinHeader_2.54mm:PinHeader_1x02_P2.54mm_Vertical" (at 208.915 77.47 0)
+      (effects (font (size 1.27 1.27)) hide)
+    )
+    (property "Datasheet" "~" (at 208.915 77.47 0)
+      (effects (font (size 1.27 1.27)) hide)
+    )
+    (pin "2")
+    (pin "1")
+    (instances
+      (project "weather_station_sensor_board"
+        (path "/204306cb-f814-4948-9295-c8792d2fccf4"
+          (reference "J6") (unit 1)
+        )
+      )
+    )
+  )
   (symbol (lib_id "power:+3V3") (at 115.57 69.85 0) (unit 1)
     (in_bom yes) (on_board yes) (dnp no)
@@
         )
       )
+    )
+  )
+  (symbol (lib_id "power:GND") (at 208.915 68.58 180) (unit 1)
+    (in_bom yes) (on_board yes) (dnp no)
+    (property "Reference" "#PWR018" (at 208.915 62.23 0)
+      (effects (font (size 1.27 1.27)) hide)
+    )
+    (property "Value" "GND" (at 208.915 62.23 0)
+      (effects (font (size 1.27 1.27)))
+    )
+    (property "Footprint" "" (at 208.915 68.58 0)
+      (effects (font (size 1.27 1.27)) hide)
+    )
+    (property "Datasheet" "" (at 208.915 68.58 0)
+      (effects (font (size 1.27 1.27)) hide)
+    )
+    (pin "1")
+    (instances
+      (project "weather_station_sensor_board"
+        (path "/204306cb-f814-4948-9295-c8792d2fccf4"
+          (reference "#PWR018") (unit 1)
+        )
+      )
